Commit message: getting jackal to run

File: simulator_setup/robot/jackal/urdf/accessories.urdf.xacro (robot description, xacro)
@@ -22,22 +22,16 @@
     - ust10            :: Hokuyo UST10
   -->
-  <xacro:if value="$(optenv JACKAL_LASER 0)">
-    <xacro:property name="lidar_model" value="$(optenv JACKAL_LASER_MODEL lms1xx)" />
+  <xacro:if value="$(optenv JACKAL_LASER 1)">
+    <xacro:property name="lidar_model" value="$(optenv JACKAL_LASER_MODEL ust10)" />
     <xacro:if value="${lidar_model == 'lms1xx'}">
       <xacro:include filename="$(find simulator_setup)/robot/jackal/urdf/accessories/sick_lms1xx_mount.urdf.xacro" />
-      <xacro:sick_lms1xx_mount prefix="$(optenv JACKAL_LASER_MOUNT front)"
-           parent_link="$(optenv JACKAL_LASER_MOUNT front)_mount"
-           topic="$(optenv JACKAL_LASER_TOPIC front/scan)">
-        <origin xyz="$(optenv JACKAL_LASER_OFFSET 0 0 0)"
-                   rpy="$(optenv JACKAL_LASER_RPY 0 0 0)" />
+      <xacro:sick_lms1xx_mount prefix="$(optenv JACKAL_LASER_MOUNT front)" parent_link="$(optenv JACKAL_LASER_MOUNT front)_mount" topic="$(optenv JACKAL_LASER_TOPIC scan)">
+        <origin xyz="$(optenv JACKAL_LASER_OFFSET 0 0 0)" rpy="$(optenv JACKAL_LASER_RPY 0 0 0)" />
       </xacro:sick_lms1xx_mount>
     </xacro:if>
     <xacro:if value="${lidar_model == 'ust10'}">
       <xacro:include filename="$(find simulator_setup)/robot/jackal/urdf/accessories/hokuyo_ust10.urdf.xacro" />
-      <xacro:hokuyo_ust10_mount prefix="$(optenv JACKAL_LASER_MOUNT front)"
-          parent_link="$(optenv JACKAL_LASER_MOUNT front)_mount"
-          topic="$(optenv JACKAL_LASER_TOPIC front/scan)">
-        <origin xyz="$(optenv JACKAL_LASER_OFFSET 0 0 0)"
-                rpy="$(optenv JACKAL_LASER_RPY 0 0 0)" />
+      <xacro:hokuyo_ust10_mount prefix="$(optenv JACKAL_LASER_MOUNT front)" parent_link="$(optenv JACKAL_LASER_MOUNT front)_mount" topic="$(optenv JACKAL_LASER_TOPIC scan)">
+        <origin xyz="$(optenv JACKAL_LASER_OFFSET 0 0 0)" rpy="$(optenv JACKAL_LASER_RPY 0 0 0)" />
       </xacro:hokuyo_ust10_mount>
     </xacro:if>
@@ -46,17 +40,11 @@
     <xacro:property name="lidar2_model" value="$(optenv JACKAL_LASER_SECONDARY_MODEL lms1xx)" />
     <xacro:if value="${lidar2_model == 'lms1xx'}">
-      <xacro:sick_lms1xx_mount prefix="$(optenv JACKAL_LASER_SECONDARY_MOUNT rear)"
-           parent_link="$(optenv JACKAL_LASER_SECONDARY_MOUNT rear)_mount"
-           topic="$(optenv JACKAL_LASER_SECONDARY_TOPIC rear/scan)">
-         <origin xyz="$(optenv JACKAL_LASER_SECONDARY_OFFSET 0 0 0)"
-                 rpy="$(optenv JACKAL_LASER_SECONDARY_RPY 0 0 3.14159)" />
-       </xacro:sick_lms1xx_mount>
+      <xacro:sick_lms1xx_mount prefix="$(optenv JACKAL_LASER_SECONDARY_MOUNT rear)" parent_link="$(optenv JACKAL_LASER_SECONDARY_MOUNT rear)_mount" topic="$(optenv JACKAL_LASER_SECONDARY_TOPIC rear/scan)">
+        <origin xyz="$(optenv JACKAL_LASER_SECONDARY_OFFSET 0 0 0)" rpy="$(optenv JACKAL_LASER_SECONDARY_RPY 0 0 3.14159)" />
+      </xacro:sick_lms1xx_mount>
     </xacro:if>
     <xacro:if value="${lidar2_model == 'ust10'}">
-      <xacro:hokuyo_ust10_mount prefix="$(optenv JACKAL_LASER_SECONDARY_MOUNT rear)"
-          parent_link="$(optenv JACKAL_LASER_SECONDARY_MOUNT rear)_mount"
-          topic="$(optenv JACKAL_LASER_SECONDARY_TOPIC rear/scan)">
-        <origin xyz="$(optenv JACKAL_LASER_SECONDARY_OFFSET 0 0 0)"
-                rpy="$(optenv JACKAL_LASER_SECONDARY_RPY 0 0 3.14159)" />
+      <xacro:hokuyo_ust10_mount prefix="$(optenv JACKAL_LASER_SECONDARY_MOUNT rear)" parent_link="$(optenv JACKAL_LASER_SECONDARY_MOUNT rear)_mount" topic="$(optenv JACKAL_LASER_SECONDARY_TOPIC rear/scan)">
+        <origin xyz="$(optenv JACKAL_LASER_SECONDARY_OFFSET 0 0 0)" rpy="$(optenv JACKAL_LASER_SECONDARY_RPY 0 0 3.14159)" />
       </xacro:hokuyo_ust10_mount>
     </xacro:if>
@@ -70,8 +58,5 @@
     <xacro:property name="lidar_3d_model" value="$(optenv JACKAL_LASER_3D_MODEL vlp16)" />
     <xacro:if value="${lidar_3d_model == 'vlp16'}">
-      <xacro:vlp16_mount
-          parent_link="$(optenv JACKAL_LASER_3D_MOUNT mid)_mount"
-          prefix="$(optenv JACKAL_LASER_3D_MOUNT mid)"
-          topic="$(optenv JACKAL_LASER_3D_TOPIC mid/points)">
+      <xacro:vlp16_mount parent_link="$(optenv JACKAL_LASER_3D_MOUNT mid)_mount" prefix="$(optenv JACKAL_LASER_3D_MOUNT mid)" topic="$(optenv JACKAL_LASER_3D_TOPIC mid/points)">
         <origin xyz="$(optenv JACKAL_LASER_3D_OFFSET 0 0 0)" rpy="$(optenv JACKAL_LASER_3D_RPY 0 0 0)" />
       </xacro:vlp16_mount>
@@ -81,6 +66,5 @@
   <xacro:if value="$(optenv JACKAL_NAVSAT 0)">
     <xacro:include filename="$(find simulator_setup)/robot/jackal/urdf/accessories/novatel_smart6.urdf.xacro" />
-    <xacro:bridge_plate mount="$(optenv JACKAL_NAVSAT_MOUNT rear)"
-                  height="$(optenv JACKAL_NAVSAT_HEIGHT 0.1)" />
+    <xacro:bridge_plate mount="$(optenv JACKAL_NAVSAT_MOUNT rear)" height="$(optenv JACKAL_NAVSAT_HEIGHT 0.1)" />
     <xacro:novatel_smart6 prefix="$(optenv JACKAL_NAVSAT_MOUNT rear)"/>
     <joint name="$(optenv JACKAL_NAVSAT_MOUNT rear)_navsat_joint" type="fixed">
@@ -95,15 +79,11 @@
   <!-- If enabled, generate the flea3 camera payload with a tilt of 30 degrees. -->
   <xacro:if value="$(optenv JACKAL_FLEA3 0)">
-    <xacro:camera_mount prefix="$(optenv JACKAL_FLEA3_MOUNT front)"
-                       tilt="$(optenv JACKAL_FLEA3_TILT 0.5236)"/>
+    <xacro:camera_mount prefix="$(optenv JACKAL_FLEA3_MOUNT front)" tilt="$(optenv JACKAL_FLEA3_TILT 0.5236)"/>
     <joint name="$(optenv JACKAL_FLEA3_MOUNT front)_camera_mount_joint" type="fixed">
-      <origin xyz="$(optenv JACKAL_FLEA3_OFFSET 0 0 0)"
-              rpy="$(optenv JACKAL_FLEA3_RPY 0 0 0)" />
+      <origin xyz="$(optenv JACKAL_FLEA3_OFFSET 0 0 0)" rpy="$(optenv JACKAL_FLEA3_RPY 0 0 0)" />
       <parent link="$(optenv JACKAL_FLEA3_MOUNT front)_mount" />
       <child link="$(optenv JACKAL_FLEA3_MOUNT front)_camera_mount" />
     </joint>
-    <xacro:pointgrey_flea3 frame="$(optenv JACKAL_FLEA3_MOUNT front)_camera" name="$(optenv JACKAL_FLEA3_NAME front)"
-      camera_x="0.0754" camera_y="0.029" camera_z="0.029"
-      camera_mass="0.085" hfov="1.0471975512" fps="60" width="640" height="512"/>
+    <xacro:pointgrey_flea3 frame="$(optenv JACKAL_FLEA3_MOUNT front)_camera" name="$(optenv JACKAL_FLEA3_NAME front)" camera_x="0.0754" camera_y="0.029" camera_z="0.029" camera_mass="0.085" hfov="1.0471975512" fps="60" width="640" height="512"/>
     <joint name="$(optenv JACKAL_FLEA3_MOUNT front)_camera_bracket_joint" type="fixed">
       <origin xyz="0.020 0 0.0245" rpy="0 0 0" />
@@ -116,15 +96,11 @@
   <!-- Disabled temporarily due to metapackage issue. -->
   <xacro:if value="$(optenv JACKAL_STEREO_FLEA3 0)">
-    <xacro:stereo_camera_mount prefix="$(optenv JACKAL_FLEA3_MOUNT front)"
-                       tilt="$(optenv JACKAL_FLEA3_TILT 0.5236)"/>
+    <xacro:stereo_camera_mount prefix="$(optenv JACKAL_FLEA3_MOUNT front)" tilt="$(optenv JACKAL_FLEA3_TILT 0.5236)"/>
     <joint name="$(optenv JACKAL_FLEA3_MOUNT front)_stereo_camera_mount_joint" type="fixed">
-      <origin xyz="$(optenv JACKAL_FLEA3_OFFSET 0 0 0)"
-              rpy="$(optenv JACKAL_FLEA3_RPY 0 0 0)" />
+      <origin xyz="$(optenv JACKAL_FLEA3_OFFSET 0 0 0)" rpy="$(optenv JACKAL_FLEA3_RPY 0 0 0)" />
       <parent link="$(optenv JACKAL_FLEA3_MOUNT front)_mount" />
       <child link="$(optenv JACKAL_FLEA3_MOUNT front)_stereo_camera_mount" />
     </joint>
-    <xacro:pointgrey_flea3 frame="$(optenv JACKAL_FLEA3_MOUNT front)_left_camera" name="$(optenv JACKAL_FLEA3_LEFT_NAME front/left)"
-      camera_x="0.0754" camera_y="0.029" camera_z="0.029"
-      camera_mass="0.085" hfov="1.0471975512" fps="60" width="640" height="512"/>
+    <xacro:pointgrey_flea3 frame="$(optenv JACKAL_FLEA3_MOUNT front)_left_camera" name="$(optenv JACKAL_FLEA3_LEFT_NAME front/left)" camera_x="0.0754" camera_y="0.029" camera_z="0.029" camera_mass="0.085" hfov="1.0471975512" fps="60" width="640" height="512"/>
     <joint name="$(optenv JACKAL_FLEA3_MOUNT front)_left_stereo_camera_bracket_joint" type="fixed">
       <origin xyz="0.015 $(optenv JACKAL_STEREO_SEPERATION 0.16) 0.0599" rpy="0 0 0" />
@@ -132,7 +108,5 @@
       <child link="$(optenv JACKAL_FLEA3_MOUNT front)_left_camera" />
     </joint>
-    <xacro:pointgrey_flea3 frame="$(optenv JACKAL_FLEA3_MOUNT front)_right_camera" name="$(optenv JACKAL_FLEA3_RIGHT_NAME front/right)"
-      camera_x="0.0754" camera_y="0.029" camera_z="0.029"
-      camera_mass="0.085" hfov="1.0471975512" fps="60" width="640" height="512"/>
+    <xacro:pointgrey_flea3 frame="$(optenv JACKAL_FLEA3_MOUNT front)_right_camera" name="$(optenv JACKAL_FLEA3_RIGHT_NAME front/right)" camera_x="0.0754" camera_y="0.029" camera_z="0.029" camera_mass="0.085" hfov="1.0471975512" fps="60" width="640" height="512"/>
     <joint name="$(optenv JACKAL_FLEA3_MOUNT front)_right_stereo_camera_bracket_joint" type="fixed">
       <origin xyz="0.015 -$(optenv JACKAL_STEREO_SEPERATION 0.16) 0.0599" rpy="0 0 0" />
@@ -146,9 +120,7 @@
   <!-- Disabled temporarily due to metapackage issue. -->
   <xacro:if value="$(optenv JACKAL_BB2 0)">
-    <xacro:camera_mount prefix="$(optenv JACKAL_BB2_MOUNT front)"
-                        tilt="$(optenv JACKAL_BB2_TILT 0)"/>
+    <xacro:camera_mount prefix="$(optenv JACKAL_BB2_MOUNT front)" tilt="$(optenv JACKAL_BB2_TILT 0)"/>
     <joint name="$(optenv JACKAL_BB2_MOUNT front)_camera_mount_joint" type="fixed">
-      <origin xyz="$(optenv JACKAL_BB2_OFFSET 0 0 0)"
-              rpy="$(optenv JACKAL_BB2_RPY 0 0 0)" />
+      <origin xyz="$(optenv JACKAL_BB2_OFFSET 0 0 0)" rpy="$(optenv JACKAL_BB2_RPY 0 0 0)" />
       <parent link="$(optenv JACKAL_BB2_MOUNT front)_mount" />
       <child link="$(optenv JACKAL_BB2_MOUNT front)_camera_mount" />
@@ -164,8 +136,5 @@
     <xacro:include filename="$(find simulator_setup)/robot/jackal/urdf/accessories/hokuyo_ust10.urdf.xacro" />
     <xacro:if value="$(optenv JACKAL_FRONT_FENDER_UST10 0)">
-      <xacro:hokuyo_ust10_mount
-        prefix="front"
-        parent_link="front_fender_accessory_link"
-        topic="$(optenv JACKAL_FRONT_LASER_TOPIC front/scan)">
+      <xacro:hokuyo_ust10_mount prefix="front" parent_link="front_fender_accessory_link" topic="$(optenv JACKAL_FRONT_LASER_TOPIC front/scan)">
         <origin xyz="0 0 0" rpy="0 0 0" />
       </xacro:hokuyo_ust10_mount>
@@ -174,8 +143,5 @@
   <xacro:if value="$(optenv JACKAL_REAR_ACCESSORY_FENDER 0)">
     <xacro:if value="$(optenv JACKAL_REAR_FENDER_UST10 0)">
-      <xacro:hokuyo_ust10_mount
-        prefix="rear"
-        parent_link="rear_fender_accessory_link"
-        topic="$(optenv JACKAL_REAR_LASER_TOPIC rear/scan)">
+      <xacro:hokuyo_ust10_mount prefix="rear" parent_link="rear_fender_accessory_link" topic="$(optenv JACKAL_REAR_LASER_TOPIC rear/scan)">
         <origin xyz="0 0 0" rpy="0 0 0" />
       </xacro:hokuyo_ust10_mount>

File: simulator_setup/robot/jackal/urdf/accessories/hokuyo_ust10.urdf.xacro (robot description, xacro)
@@ -2,18 +2,15 @@
 <robot xmlns:xacro="http://ros.org/wiki/xacro">
   <xacro:macro name="hokuyo_ust10_mount" params="prefix topic parent_link *origin">
-    <xacro:macro name="hokuyo_ust10" params="frame:=laser topic:=scan sample_size:=720 update_rate:=50
-               min_angle:=-2.35619 max_angle:=2.35619 min_range:=0.1 max_range:=30.0 robot_namespace:=/">
+    <xacro:macro name="hokuyo_ust10" params="frame:=laser topic:=scan sample_size:=720 update_rate:=50 min_angle:=-2.35619 max_angle:=2.35619 min_range:=0.1 max_range:=30.0 robot_namespace:=/">
       <link name="${frame}">
         <inertial>
           <mass value="1.1" />
           <origin xyz="0 0 0" />
-          <inertia ixx="${0.0833333 * 1.1 * (0.102*0.102 + 0.152*0.152)}" ixy="0.0" ixz="0.0"
-            iyy="${0.0833333 * 1.1 * (0.105*0.105 + 0.152*0.152)}" iyz="0.0"
-            izz="${0.0833333 * 1.1 * (0.105*0.105 + 0.102*0.102)}" />
+          <inertia ixx="${0.0833333 * 1.1 * (0.102*0.102 + 0.152*0.152)}" ixy="0.0" ixz="0.0" iyy="${0.0833333 * 1.1 * (0.105*0.105 + 0.152*0.152)}" iyz="0.0" izz="${0.0833333 * 1.1 * (0.105*0.105 + 0.102*0.102)}" />
         </inertial>
       </link>
       <gazebo reference="${frame}">
         <turnGravityOff>true</turnGravityOff>
-        <sensor type="ray" name="${frame}">
+        <sensor type="gpu_ray" name="${frame}">
           <pose>0 0 0 0 0 0</pose>
           <visualize>false</visualize>
@@ -39,5 +36,5 @@
             </noise>
           </ray>
-          <plugin name="gazebo_ros_laser" filename="libgazebo_ros_laser.so">
+          <plugin name="gazebo_ros_laser" filename="libgazebo_ros_gpu_laser.so">
             <topicName>${topic}</topicName>
             <frameName>${frame}</frameName>
