Commit message: added eval csv for guldenring and navrep

File: simulator_setup/robot/rto/urdf/components/rto_parts.urdf.xacro (robot description, xacro)
@@ -53,10 +53,10 @@
                 <inertia ixx="1.0" ixy="0.0" ixz="0.0" iyy="1.0" iyz="0.0" izz="1.0"/>
             </inertial>
-            <collision>
+            <!-- <collision>
                 <origin xyz="0 0 0" rpy="0 0 0"/>
                 <geometry>
                     <box size="0.25 0.11 0.16"/>
                 </geometry>
-            </collision>
+            </collision> -->
         </link>
         <joint name="${name}_joint" type="fixed">

File: simulator_setup/robot/rto/urdf/components/rto_platform.urdf (robot description, URDF)
Before this commit: robot rto, 7 links, 6 joints
Links:
- link command_bridge_link: geometry 

File: simulator_setup/robot/rto/urdf/components/rto_platform_kinect.urdf (robot description, URDF)
Before this commit: robot rto, 8 links, 7 joints
Links:
- link base_link: geometry visual mesh filename=package://simulator_setup/robot/rto/meshes/parts/rto_base.d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 scale=0.01 0.01 0.01
- link command_bridge_link: geometry 
- link kinect_link: geometry visual mesh filename=package://simulator_setup/robot/rto/meshes/sensors/kinect.d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

Commit message: added basic: waffle_pi, rto, tiago

File: simulator_setup/robot/rto/urdf/components/rto_parts.urdf.xacro (robot description, xacro)
@@ -53,10 +53,10 @@
                 <inertia ixx="1.0" ixy="0.0" ixz="0.0" iyy="1.0" iyz="0.0" izz="1.0"/>
             </inertial>
-            <!-- <collision>
+            <collision>
                 <origin xyz="0 0 0" rpy="0 0 0"/>
                 <geometry>
                     <box size="0.25 0.11 0.16"/>
                 </geometry>
-            </collision> -->
+            </collision>
         </link>
         <joint name="${name}_joint" type="fixed">

File: simulator_setup/robot/rto/urdf/components/rto_platform.urdf (robot description, URDF)
Before this commit: robot rto, 7 links, 6 joints
Links:
- link command_bridge_link: geometry collision box size=0.25 0.11 0.16

File: simulator_setup/robot/rto/urdf/components/rto_platform_kinect.urdf (robot description, URDF)
Before this commit: robot rto, 8 links, 7 joints
Links:
- link base_link: geometry collision cylinder length=0.05 radius=0.18; visual mesh filename=package://simulator_setup/robot/rto/meshes/parts/rto_base.d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 scale=0.01 0.01 0.01
- link command_bridge_link: geometry collision box size=0.25 0.11 0.16
- link kinect_link: geometry collision box size=0.064 0.121 0.0381; visual mesh filename=package://simulator_setup/robot/rto/meshes/sensors/kinect.d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

File: simulator_setup/robot/rto/urdf/rto.urdf.xacro (robot description, xacro)
@@ -1,11 +1,6 @@
 <?xml version="1.0"?>
 <robot name="rto" xmlns:xacro="http://wiki.ros.org/xacro">
-  <xacro:property name="PI" value="3.1415926535897931" />
   <xacro:include filename="$(find simulator_setup)/robot/rto/urdf/components/rto_parts.urdf.xacro"/>
   <xacro:include filename="$(find simulator_setup)/robot/rto/urdf/components/rto_body.urdf.xacro"/>
-  <xacro:include filename="$(find simulator_setup)/robot/rto/urdf/sensors/hokuyo.urdf.xacro" />
-  <xacro:hokuyo_ust-10lx_mount prefix="front"
-                                topic="scan"
-                                location="1" />
   <xacro:rto_body/>
 </robot>

File: simulator_setup/robot/rto/urdf/sensors/asus_xtion_pro.urdf.xacro (robot description, xacro)
@@ -1,5 +1,5 @@
 <?xml version="1.0"?>
 <robot name="sensor_asus_xtion_pro" xmlns:xacro="http://ros.org/wiki/xacro">
-  <xacro:include filename="$(find rto_description)/urdf/sensors/3dsensor_gazebo.urdf.xacro"/>
+  <xacro:include filename="$(find simulator_setup)/robot/rto/urdf/sensors/3dsensor_gazebo.urdf.xacro"/>
   <xacro:property name="M_SCALE2" value="0.001"/>
   <xacro:property name="asus_xtion_pro_depth_rel_rgb_py" value="0.0270" />

File: simulator_setup/robot/rto/urdf/sensors/hokuyo.urdf.xacro (robot description, xacro)
@@ -1,51 +1,58 @@
 <?xml version="1.0"?>
-<robot xmlns:xacro="http://ros.org/wiki/xacro">
-  <xacro:macro name="hokuyo_ust-10lx_mount" params="prefix topic location">
-    <joint name="${prefix}_laser_joint" type="fixed">
-      <origin xyz="${location * 0.3932} 0 0.2330" rpy="0 0 ${PI/2 - (location * PI/2)}" />
-      <parent link="base_link" />
-      <child link="${prefix}_laser" />
+<root xmlns:xacro="http://www.ros.org/wiki/xacro">
+  <xacro:property name="M_PI" value="3.14159"/>
+  <xacro:property name="M_SCALE" value="0.01"/>
+  <xacro:property name="HOKUYO_RADIUS" value="0.02"/>
+  <xacro:property name="HOKUYO_LENGTH" value="0.07"/>
+  <xacro:macro name="hokuyo" params="parent name *origin">
+    <joint name="${name}_joint" type="fixed">
+      <xacro:insert_block name="origin" />
+      <parent link="${parent}"/>
+      <child link="${name}_link" />
     </joint>
-    <link name="${prefix}_laser">
+    <link name="${name}_link">
       <inertial>
-        <mass value="0.130" />
+        <mass value="0.00001" />
         <origin xyz="0 0 0" />
-        <inertia ixx="${0.0833333 * 0.130 * (0.05*0.05 + 0.07*0.07)}" ixy="0.0" ixz="0.0"
-          iyy="${0.0833333 * 0.130 * (0.05*0.05 + 0.07*0.07)}" iyz="0.0"
-          izz="${0.0833333 * 0.130 * (0.05*0.05 + 0.05*0.05)}" />
+        <inertia ixx="1.0" ixy="0.0" ixz="0.0"
+		 iyy="1.0" iyz="0.0"
+		 izz="1.0" />
       </inertial>
       <visual>
-        <origin xyz="0 0 0" rpy="0 0 0" />
+        <origin xyz="0 0 -0.05" rpy="0 0 ${M_PI/2}" />
         <geometry>
-          <!-- Origin of this mesh is the focal point of the LIDAR. -->
-          <mesh filename="package://simulator_setup/robot/pepper/meshes/ust-10lx.stl" />
+          <mesh filename="package://simulator_setup/robot/rto/meshes/sensors/hokuyo.dae" scale="${M_SCALE} ${M_SCALE} ${M_SCALE}"/>
         </geometry>
-        <material name="dark_grey" />
       </visual>
       <collision>
-        <origin xyz="0 0 -0.0122" rpy="0 0 0" />
+        <origin xyz="0 0 ${HOKUYO_LENGTH/2}" rpy="0 0 0" />
         <geometry>
-          <box size="0.05 0.05 0.07" />
+          <cylinder radius="${HOKUYO_RADIUS}" length="${HOKUYO_LENGTH}" />
         </geometry>
       </collision>
     </link>
-    <gazebo reference="${prefix}_laser">
-      <turnGravityOff>false</turnGravityOff>
-      <sensor type="ray" name="${prefix}_laser">
+    <!-- gazebo extensions -->
+    <xacro:hokuyo_gazebo name="${name}" ros_topic="scan" update_rate="10" min_angle="-1.570796" max_angle="1.570796"/>
+  </xacro:macro>
+  <!--GAZEBO PLUGIN-->
+  <xacro:macro name="hokuyo_gazebo" params="name ros_topic update_rate min_angle max_angle">
+    <gazebo reference="${name}_link">
+      <sensor name="${name}" type="gpu_ray">
+        <!--always_on>true</always_on-->
+        <update_rate>40</update_rate>
         <pose>0 0 0 0 0 0</pose>
         <visualize>false</visualize>
-        <update_rate>50</update_rate>
         <ray>
           <scan>
             <horizontal>
-              <samples>1080</samples>
-              <resolution>1</resolution>
-              <min_angle>0</min_angle>
-              <max_angle>6.28319</max_angle>
+              <samples>683</samples>
+              <resolution>0.36</resolution>
+              <min_angle>-2,0944</min_angle>
+              <max_angle>2,0944</max_angle>
             </horizontal>
           </scan>
           <range>
-            <min>0.20</min>
-            <max>25.0</max>
+            <min>0.03</min>
+            <max>5.6</max>
             <resolution>0.01</resolution>
           </range>
@@ -53,15 +60,13 @@
             <type>gaussian</type>
             <mean>0.0</mean>
-            <stddev>0.001</stddev>
+            <stddev>0.005</stddev>
           </noise>
         </ray>
-        <plugin name="gazebo_ros_laser" filename="libgazebo_ros_laser.so">
-          <topicName>${topic}</topicName>
-          <frameName>${prefix}_laser</frameName>
-          <hokuyoMinIntensity>101</hokuyoMinIntensity>
+        <plugin name="gazebo_ros_${name}_controller" filename="libgazebo_ros_gpu_laser.so">
+          <topicName>${ros_topic}</topicName>
+          <frameName>${name}_link</frameName>
         </plugin>
       </sensor>
-      <material>Gazebo/DarkGrey</material>
     </gazebo>
   </xacro:macro>
-</robot>
+</root>

File: simulator_setup/robot/rto/urdf/sensors/realsense_d415.urdf.xacro (robot description, xacro)
@@ -8,6 +8,6 @@
 <robot name="sensor_d415" xmlns:xacro="http://ros.org/wiki/xacro">
   <!-- Includes -->
-  <xacro:include filename="$(find realsense2_description)/urdf/_materials.urdf.xacro" />
-  <xacro:include filename="$(find realsense2_description)/urdf/_usb_plug.urdf.xacro" />
+  <xacro:include filename="$(find simulator_setup)/robot/rto/realsense2/urdf/_materials.urdf.xacro" />
+  <xacro:include filename="$(find simulator_setup)/robot/rto/realsense2/urdf/_usb_plug.urdf.xacro" />
   <xacro:macro name="sensor_d415" params="parent *origin  name:=camera  use_nominal_extrinsics:=false  add_plug:=false">
     <xacro:property name="M_PI" value="3.1415926535897931" />
@@ -46,5 +46,5 @@
         <geometry>
           <!-- <box size="${d415_cam_width} ${d415_cam_height} ${d415_cam_depth}"/> -->
-	         <mesh filename="package://realsense2_description/meshes/d415.stl" />
+	         <mesh filename="package://simulator_setup/robot/rto/realsense2/meshes/d415.stl" />
         </geometry>
         <material name="aluminum"/>
